File: Hardware/Door_lock.kicad_pcb (KiCad board)
At the start: 2 copper layers, 56 parts, among them J1 Conn_02x05_Odd_Even, J10 Conn_01x02_Pin, J2 Conn_01x02, J3 Conn_01x02, J4 Conn_01x02, J5 Conn_01x02, J6 Conn_01x02, J7 Conn_01x02, J8 Conn_01x02, J9 Conn_01x02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

Commit message: update hardware design
Parts:
- removed C2: 20pF, Capacitor_SMD:C_0603_1608Metric
- removed J10: Conn_01x02_Pin, TerminalBlock:TerminalBlock_bornier-2_P5.08mm
- removed Y1: 24MHz, LOKAL:OSC-SMD_4P-L3.2-W2.5-BL
- added Address: SW_DIP_x05, Button_Switch_THT:SW_DIP_SPSTx05_Slide_9.78x14.88mm_W7.62mm_P2.54mm, F.Cu at (65.5, 85.2)
- added D4: ESD9B5.0ST5G, Diode_SMD:D_SMB, F.Cu at (95.9, 76.5)
- added D5: ESD9B5.0ST5G, Diode_SMD:D_SMB, F.Cu at (95.9, 65.0)
- added H3: MountingHole, MountingHole:MountingHole_3.2mm_M3_Pad_Via, F.Cu at (32.2, 41.5)
- added H4: MountingHole, MountingHole:MountingHole_3.2mm_M3_Pad_Via, F.Cu at (108.7, 83.1)
- added R10: 560, Resistor_SMD:R_0603_1608Metric, F.Cu at (82.1, 71.5)
- added R12: 120, Resistor_SMD:R_0603_1608Metric, F.Cu at (95.9, 70.8)
- added R13: 10, Resistor_SMD:R_0603_1608Metric, F.Cu at (93.5, 70.0)
- added R14: 10, Resistor_SMD:R_0603_1608Metric, F.Cu at (93.5, 71.6)
- added RN1: R_Network05, Resistor_SMD:R_Array_Convex_5x0603, F.Cu at (80.7, 80.3)
- added RS485: Conn_01x04, TerminalBlock_Phoenix:TerminalBlock_Phoenix_MKDS-1,5-4-5.08_1x04_P5.08mm_Horizontal, F.Cu at (33.8, 60.6)
- added RS485: Conn_01x04, TerminalBlock_Phoenix:TerminalBlock_Phoenix_MKDS-1,5-4-5.08_1x04_P5.08mm_Horizontal, F.Cu at (106.9, 75.8)
- added U9: MAX485E, Package_SO:SOIC-8-1EP_3.9x4.9mm_P1.27mm_EP2.62x3.51mm_ThermalVias, F.Cu at (87.6, 70.8)
- C1: value 20pF -> 100nF
- FB1: renamed from J6; footprint Connector_PinHeader_2.54mm:PinHeader_2x01_P2.54mm_Vertical -> Connector_JST:JST_XH_B2B-XH-A_1x02_P2.50mm_Vertical
- FB2: renamed from J7; footprint Connector_PinHeader_2.54mm:PinHeader_2x01_P2.54mm_Vertical -> Connector_JST:JST_XH_B2B-XH-A_1x02_P2.50mm_Vertical
- FB3: renamed from J8; footprint Connector_PinHeader_2.54mm:PinHeader_2x01_P2.54mm_Vertical -> Connector_JST:JST_XH_B2B-XH-A_1x02_P2.50mm_Vertical
- FB4: renamed from J9; footprint Connector_PinHeader_2.54mm:PinHeader_2x01_P2.54mm_Vertical -> Connector_JST:JST_XH_B2B-XH-A_1x02_P2.50mm_Vertical
- O1: renamed from J4; footprint Connector_PinHeader_2.54mm:PinHeader_2x01_P2.54mm_Vertical -> Connector_JST:JST_XH_B2B-XH-A_1x02_P2.50mm_Vertical
- O2: renamed from J2; footprint Connector_PinHeader_2.54mm:PinHeader_2x01_P2.54mm_Vertical -> Connector_JST:JST_XH_B2B-XH-A_1x02_P2.50mm_Vertical
- O3: renamed from J3; footprint Connector_PinHeader_2.54mm:PinHeader_2x01_P2.54mm_Vertical -> Connector_JST:JST_XH_B2B-XH-A_1x02_P2.50mm_Vertical
- O4: renamed from J5; footprint Connector_PinHeader_2.54mm:PinHeader_2x01_P2.54mm_Vertical -> Connector_JST:JST_XH_B2B-XH-A_1x02_P2.50mm_Vertical
- R11, R4, R7, R9: moved to B.Cu
- moved R21 91.5 mm to (103.7, 47.1)
- moved R22 88.5 mm to (102.2, 47.1), turned to -90 degrees
- moved FB4 87.9 mm to (101.3, 41.5)
- moved R9 78.7 mm to (96.4, 44.8), turned to 0 degrees
- moved R8 77.7 mm to (97.2, 56.3)
- moved U7 77.6 mm to (97.2, 54.3), turned to 90 degrees
- moved O4 73.1 mm to (92.8, 41.5), turned to 180 degrees
- moved Q3 67.3 mm to (92.0, 52.0), turned to -90 degrees
- moved H2 66.7 mm to (32.2, 83.1)
- moved WCH-LINK 55.0 mm to (44.2, 84.7), turned to 90 degrees
- moved R2 47.0 mm to (84.6, 83.1)
- moved D1 46.8 mm to (84.6, 84.9)
- moved H1 38.9 mm to (108.5, 41.5)
- moved FB3 38.7 mm to (84.3, 41.5)
- moved R19 37.4 mm to (87.0, 47.1), turned to 90 degrees
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- renumbered J1 to WCH-LINK
Connections:
- C1 pad 2: Net-(U1-PA1/OSCI/A1) -> +5V
- U1 pad 10: FB4 -> IO3
- U1 pad 11: IO4 -> FB2
- U1 pad 12: IO3 -> IO2
- U1 pad 13: IO2 -> FB1
- U1 pad 16: unconnected-(U1-PD2/A3/T1CH1/T2CH3_-Pad16) -> addr1
- U1 pad 17: unconnected-(U1-PD3/A4/T2CH2/AETR-Pad17) -> addr2
- U1 pad 2: Net-(U1-PA1/OSCI/A1) -> addr3
- U1 pad 3: Net-(U1-PA2/OSCO/A0/T1CH2N) -> addr4
- U1 pad 5: unconnected-(U1-PD0/T1CH1N/OPN1-Pad5) -> addr5
- U1 pad 7: FB1 -> FB4
- U1 pad 8: FB2 -> IO4
- WCH-LINK pad 7: TX -> unconnected-(J1-Pin_7-Pad7)
- WCH-LINK pad 9: RX -> unconnected-(J1-Pin_9-Pad9)
Routing:
- net +3V3: track 0.00 -> 211.5 mm, vias 0 -> 10
- net +12V: track 0.00 -> 154.6 mm, vias 0 -> 4
- net A: track 0.00 -> 92.5 mm
- net B: track 0.00 -> 91.2 mm
- net +5V: track 0.00 -> 73.9 mm, vias 0 -> 2
- net FB4: track 0.00 -> 42.3 mm
- net FB1: track 0.00 -> 34.8 mm
- net PD4: track 0.00 -> 34.5 mm, vias 0 -> 2
- net IO4: track 0.00 -> 33.7 mm
- net addr1: track 0.00 -> 31.8 mm
- net IO1: track 0.00 -> 31.5 mm
- net SWDIO: track 0.00 -> 30.9 mm
- net FB3: track 0.00 -> 26.4 mm
- net addr2: track 0.00 -> 25.5 mm
- net TX: track 0.00 -> 20.6 mm, vias 0 -> 2
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- added copper zone on B.Cu, net GND
- added copper zone on F.Cu, net GND
- added copper zone on F.Cu, net Net-(D2-K)
Other:
- board outline added: 84.8 x 49.7 mm
- copper layers 2 -> 4
- rule pad_to_mask_clearance: 0 -> 0.01
