File: Hardware/Door_lock.kicad_sch (KiCad schematic)
At the start: 56 parts, among them J1 Conn_02x05_Odd_Even, J10 Conn_01x02_Pin, J2 Conn_01x02, J3 Conn_01x02, J4 Conn_01x02, J5 Conn_01x02, J6 Conn_01x02, J7 Conn_01x02, J8 Conn_01x02, J9 Conn_01x02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

Commit message: update hardware design
Parts:
- removed C2: 20pF, Capacitor_SMD:C_0603_1608Metric, symbol Device:C
- removed J10: Conn_01x02_Pin, TerminalBlock:TerminalBlock_bornier-2_P5.08mm, symbol Connector:Conn_01x02_Pin
- removed Y1: 24MHz, LOKAL:OSC-SMD_4P-L3.2-W2.5-BL, symbol Device:Crystal_GND24_Small
- added D4, D5: ESD9B5.0ST5G, Diode_SMD:D_SMB, symbol Diode:ESD9B5.0ST5G
- added H3, H4: MountingHole, MountingHole:MountingHole_3.2mm_M3_Pad_Via, symbol Mechanical:MountingHole
- added J11, J12: Conn_01x04, TerminalBlock_Phoenix:TerminalBlock_Phoenix_MKDS-1,5-4-5.08_1x04_P5.08mm_Horizontal, symbol Connector_Generic:Conn_01x04
- added R10: 560, Resistor_SMD:R_0603_1608Metric, symbol Device:R
- added R12: 120, Resistor_SMD:R_0603_1608Metric, symbol Device:R
- added R13, R14: 10, Resistor_SMD:R_0603_1608Metric, symbol Device:R
- added RN1: R_Network05, Resistor_SMD:R_Array_Convex_5x0603, symbol Device:R_Network05
- added SW1: SW_DIP_x05, Button_Switch_THT:SW_DIP_SPSTx05_Slide_9.78x14.88mm_W7.62mm_P2.54mm, symbol Switch:SW_DIP_x05
- added U9: MAX485E, Package_SO:SOIC-8-1EP_3.9x4.9mm_P1.27mm_EP2.62x3.51mm_ThermalVias, symbol Interface_UART:MAX485E
- C1: value 20pF -> 100nF
- J2, J3, J4, J5, J6, J7, J8, J9: footprint Connector_PinHeader_2.54mm:PinHeader_2x01_P2.54mm_Vertical -> Connector_JST:JST_XH_B2B-XH-A_1x02_P2.50mm_Vertical
Connections:
- net +12V: now also J11.1 (Pin_1), J12.4 (Pin_4)
- net +3V3: now also RN1.1 (common)
- net +5V: now also C1.2, U9.8 (VCC)
- net FB1: now also U1.13 (PC6/MOSI/T1CH1CH3N_); no longer U1.7 (PC0/T2CH3/UTX_)
- net FB2: now also U1.11 (PC4/A2/T1CH4/MCO); no longer U1.8 (PC1/SDA/NSS/T2CH4_)
- net FB4: now also U1.7 (PC0/T2CH3/UTX_); no longer U1.10 (PC3/T1CH3/T1CH1N_)
- net GND: now also D4.2 (A2), D5.2 (A2), J11.2 (Pin_2), J12.3 (Pin_3), SW1.1, SW1.2, SW1.3, SW1.4, SW1.5, U9.5 (GND)
- net IO2: now also U1.12 (PC5/SCK/T1ETR/T2CH1ETR_); no longer U1.13 (PC6/MOSI/T1CH1CH3N_)
- net IO3: now also U1.10 (PC3/T1CH3/T1CH1N_); no longer U1.12 (PC5/SCK/T1ETR/T2CH1ETR_)
- net IO4: now also U1.8 (PC1/SDA/NSS/T2CH4_); no longer U1.11 (PC4/A2/T1CH4/MCO)
- net PD4: now also R10.1
- net RX: now also U9.1 (RO); no longer J1.9 (Pin_9)
- net TX: now also U9.4 (DI); no longer J1.7 (Pin_7)
- net addr1: now reaches U1.16 (PD2/A3/T1CH1/T2CH3_)
- net addr1: now also RN1.6 (R5), SW1.10
- net addr2: now reaches U1.17 (PD3/A4/T2CH2/AETR)
- net addr2: now also RN1.5 (R4), SW1.9
- net addr3: now reaches U1.2 (PA1/OSCI/A1)
- net addr3: now also RN1.4 (R3), SW1.8; no longer C1.2
- net addr4: now reaches U1.3 (PA2/OSCO/A0/T1CH2N)
- net addr4: now also RN1.3 (R2), SW1.7
- net addr5: now reaches U1.5 (PD0/T1CH1N/OPN1)
- net addr5: now also RN1.2 (R1), SW1.6
- new net: R14.2, U9.6 (A)
- new net: R10.2, U9.2 (~{RE}), U9.3 (DE)
- new net: R13.2, U9.7 (B)
- new net A: D4.1 (A1), J11.4 (Pin_4), J12.1 (Pin_1), R12.1, R14.1
- new net B: D5.1 (A1), J11.3 (Pin_3), J12.2 (Pin_2), R12.2, R13.1
- no-connect marks 8 -> 7
Other:
- moved on the sheet: H1, H2, J1, J2, J3, J4, J5, J6, J7, J8, J9, Q1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
